Commit message: feat: use source MentorPi mecanum model

File: ros2_ws/src/mentorpi_gz_sim/models/mentorpi_m1/model.sdf.xacro (robot description, xacro)
@@ -4,6 +4,4 @@
   <xacro:property name="robot_name" value="$(arg robot_name)"/>
   <xacro:property name="wheel_radius" value="0.032"/>
-  <xacro:property name="wheel_x" value="0.070"/>
-  <xacro:property name="wheel_y" value="0.094"/>
   <model name="${robot_name}" canonical_link="base_footprint">
     <link name="base_footprint">
@@ -16,7 +14,7 @@
         <material><ambient>0.04 0.28 0.62 1</ambient><diffuse>0.04 0.28 0.62 1</diffuse></material></visual>
     </link>
-    <xacro:macro name="wheel" params="name x y friction_x friction_y">
+    <xacro:macro name="wheel" params="name x y z friction_x friction_y">
       <link name="${name}_wheel">
-        <pose>${x} ${y} ${wheel_radius} -1.5708 0 0</pose>
+        <pose>${x} ${y} ${z} -1.5708 0 0</pose>
         <inertial><mass>0.05</mass><inertia><ixx>0.00002</ixx><ixy>0</ixy><ixz>0</ixz><iyy>0.00002</iyy><iyz>0</iyz><izz>0.00002</izz></inertia></inertial>
         <collision name="collision"><geometry><sphere><radius>${wheel_radius}</radius></sphere></geometry>
@@ -31,31 +29,31 @@
       </joint>
     </xacro:macro>
-    <xacro:wheel name="front_left" x="${wheel_x}" y="${wheel_y}" friction_x="1" friction_y="-1"/>
-    <xacro:wheel name="front_right" x="${wheel_x}" y="-${wheel_y}" friction_x="1" friction_y="1"/>
-    <xacro:wheel name="back_left" x="-${wheel_x}" y="${wheel_y}" friction_x="1" friction_y="1"/>
-    <xacro:wheel name="back_right" x="-${wheel_x}" y="-${wheel_y}" friction_x="1" friction_y="-1"/>
-    <link name="base_laser"><pose>-0.012242 -0.00008533 0.162501 0 0 0</pose>
+    <xacro:wheel name="front_left" x="0.067052" y="0.07591" z="0.051592" friction_x="1" friction_y="-1"/>
+    <xacro:wheel name="front_right" x="0.067052" y="-0.07591" z="0.051592" friction_x="1" friction_y="1"/>
+    <xacro:wheel name="back_left" x="-0.06764" y="0.07591" z="0.051586" friction_x="1" friction_y="1"/>
+    <xacro:wheel name="back_right" x="-0.067621" y="-0.07591" z="0.051592" friction_x="1" friction_y="-1"/>
+    <link name="lidar_frame"><pose>-0.012242 -0.00008533 0.162501 0 0 0</pose>
       <inertial><mass>0.05</mass><inertia><ixx>0.00001</ixx><ixy>0</ixy><ixz>0</ixz><iyy>0.00001</iyy><iyz>0</iyz><izz>0.00001</izz></inertia></inertial>
       <visual name="visual"><geometry><cylinder><radius>0.032</radius><length>0.025</length></cylinder></geometry></visual>
       <sensor name="lidar" type="gpu_lidar">
         <always_on>true</always_on><update_rate>12</update_rate><visualize>false</visualize>
-        <topic>/${robot_name}/scan_raw</topic><gz_frame_id>${robot_name}/base_laser</gz_frame_id>
+        <topic>/${robot_name}/scan_raw</topic><gz_frame_id>${robot_name}/lidar_frame</gz_frame_id>
         <lidar><scan><horizontal><samples>360</samples><resolution>1</resolution><min_angle>-3.14159</min_angle><max_angle>3.14159</max_angle></horizontal></scan>
           <range><min>0.08</min><max>12.0</max><resolution>0.01</resolution></range></lidar>
       </sensor>
     </link>
-    <joint name="laser_joint" type="fixed"><parent>base_footprint</parent><child>base_laser</child></joint>
-    <link name="depth_camera_link"><pose>0.061376 -0.00013463 0.121154 0 0 0</pose>
+    <joint name="lidar_Joint" type="fixed"><parent>base_footprint</parent><child>lidar_frame</child></joint>
+    <link name="depth_cam"><pose>0.061376 -0.00013463 0.121154 0 0 0</pose>
       <inertial><mass>0.08</mass><inertia><ixx>0.00002</ixx><ixy>0</ixy><ixz>0</ixz><iyy>0.00002</iyy><iyz>0</iyz><izz>0.00002</izz></inertia></inertial>
       <visual name="visual"><geometry><box><size>0.045 0.055 0.025</size></box></geometry></visual>
       <sensor name="depth_camera" type="depth_camera">
         <always_on>true</always_on><update_rate>10</update_rate><visualize>false</visualize>
-        <topic>/${robot_name}/depth/image_raw</topic><gz_frame_id>${robot_name}/depth_camera_link</gz_frame_id>
+        <topic>/${robot_name}/depth/image_raw</topic><gz_frame_id>${robot_name}/depth_cam</gz_frame_id>
         <camera><horizontal_fov>1.047</horizontal_fov><image><width>320</width><height>240</height><format>R8G8B8</format></image>
           <camera_info_topic>/${robot_name}/depth/camera_info</camera_info_topic><clip><near>0.10</near><far>8.0</far></clip></camera>
       </sensor>
     </link>
-    <joint name="depth_camera_joint" type="fixed"><parent>base_footprint</parent><child>depth_camera_link</child></joint>
-    <link name="imu_link"><pose>0 0 0.105 0 0 0</pose>
+    <joint name="cam_Joint" type="fixed"><parent>base_footprint</parent><child>depth_cam</child></joint>
+    <link name="imu_link"><pose>0 0 0.07 0 0 0</pose>
       <inertial><mass>0.01</mass><inertia><ixx>0.000001</ixx><ixy>0</ixy><ixz>0</ixz><iyy>0.000001</iyy><iyz>0</iyz><izz>0.000001</izz></inertia></inertial>
       <sensor name="imu" type="imu"><always_on>true</always_on><update_rate>50</update_rate>
@@ -66,5 +64,5 @@
       <front_left_joint>front_left_wheel_joint</front_left_joint><front_right_joint>front_right_wheel_joint</front_right_joint>
       <back_left_joint>back_left_wheel_joint</back_left_joint><back_right_joint>back_right_wheel_joint</back_right_joint>
-      <wheelbase>0.140</wheelbase><wheel_separation>0.188</wheel_separation><wheel_radius>${wheel_radius}</wheel_radius>
+      <wheelbase>0.13468</wheelbase><wheel_separation>0.15182</wheel_separation><wheel_radius>${wheel_radius}</wheel_radius>
       <odom_publish_frequency>30</odom_publish_frequency><topic>/${robot_name}/controller/cmd_vel</topic>
       <odom_topic>/${robot_name}/odom</odom_topic><tf_topic>/${robot_name}/tf</tf_topic>

Commit message: feat: add configurable MentorPi forklift model

File: ros2_ws/src/mentorpi_gz_sim/models/mentorpi_m1/model.sdf.xacro (robot description, xacro)
@@ -4,4 +4,5 @@
   <xacro:property name="robot_name" value="$(arg robot_name)"/>
   <xacro:property name="wheel_radius" value="0.032"/>
+  <xacro:include filename="$(find mentorpi_description)/urdf/forklift_camera_config.xacro"/>
   <model name="${robot_name}" canonical_link="base_footprint">
     <link name="base_footprint">
@@ -33,4 +34,32 @@
     <xacro:wheel name="back_left" x="-0.06764" y="0.07591" z="0.051586" friction_x="1" friction_y="1"/>
     <xacro:wheel name="back_right" x="-0.067621" y="-0.07591" z="0.051592" friction_x="1" friction_y="-1"/>
+    <link name="fork_mast"><pose>0.115 0 0.18 0 0 0</pose>
+      <inertial><mass>0.20</mass><inertia><ixx>0.0018</ixx><ixy>0</ixy><ixz>0</ixz><iyy>0.0018</iyy><iyz>0</iyz><izz>0.0001</izz></inertia></inertial>
+      <collision name="collision"><geometry><box><size>0.026 0.12 0.30</size></box></geometry></collision>
+      <visual name="visual"><geometry><box><size>0.026 0.12 0.30</size></box></geometry>
+        <material><ambient>0.04 0.04 0.04 1</ambient><diffuse>0.04 0.04 0.04 1</diffuse></material></visual>
+    </link>
+    <joint name="fork_mast_joint" type="fixed"><parent>base_footprint</parent><child>fork_mast</child></joint>
+    <link name="fork_carriage"><pose>0.115 0 0.025 0 0 0</pose>
+      <inertial><mass>0.10</mass><inertia><ixx>0.0003</ixx><ixy>0</ixy><ixz>0</ixz><iyy>0.0001</iyy><iyz>0</iyz><izz>0.0003</izz></inertia></inertial>
+      <collision name="collision"><pose>0 0 0.045 0 0 0</pose><geometry><box><size>0.030 0.13 0.09</size></box></geometry></collision>
+      <visual name="visual"><pose>0 0 0.045 0 0 0</pose><geometry><box><size>0.030 0.13 0.09</size></box></geometry>
+        <material><ambient>0.04 0.04 0.04 1</ambient><diffuse>0.04 0.04 0.04 1</diffuse></material></visual>
+    </link>
+    <joint name="fork_carriage_joint" type="prismatic"><parent>base_footprint</parent><child>fork_carriage</child>
+      <axis><xyz>0 0 1</xyz><limit><lower>0.0</lower><upper>0.11</upper><effort>20</effort><velocity>0.05</velocity></limit></axis>
+    </joint>
+    <link name="fork_left"><pose relative_to="fork_carriage">0.09 0.05 0 0 0 0</pose>
+      <inertial><mass>0.03</mass><inertia><ixx>0.00001</ixx><ixy>0</ixy><ixz>0</ixz><iyy>0.00008</iyy><iyz>0</iyz><izz>0.00008</izz></inertia></inertial>
+      <collision name="collision"><geometry><box><size>0.18 0.014 0.010</size></box></geometry></collision>
+      <visual name="visual"><geometry><box><size>0.18 0.014 0.010</size></box></geometry><material><ambient>0.04 0.04 0.04 1</ambient><diffuse>0.04 0.04 0.04 1</diffuse></material></visual>
+    </link>
+    <joint name="fork_left_joint" type="fixed"><parent>fork_carriage</parent><child>fork_left</child></joint>
+    <link name="fork_right"><pose relative_to="fork_carriage">0.09 -0.05 0 0 0 0</pose>
+      <inertial><mass>0.03</mass><inertia><ixx>0.00001</ixx><ixy>0</ixy><ixz>0</ixz><iyy>0.00008</iyy><iyz>0</iyz><izz>0.00008</izz></inertia></inertial>
+      <collision name="collision"><geometry><box><size>0.18 0.014 0.010</size></box></geometry></collision>
+      <visual name="visual"><geometry><box><size>0.18 0.014 0.010</size></box></geometry><material><ambient>0.04 0.04 0.04 1</ambient><diffuse>0.04 0.04 0.04 1</diffuse></material></visual>
+    </link>
+    <joint name="fork_right_joint" type="fixed"><parent>fork_carriage</parent><child>fork_right</child></joint>
     <link name="lidar_frame"><pose>-0.012242 -0.00008533 0.162501 0 0 0</pose>
       <inertial><mass>0.05</mass><inertia><ixx>0.00001</ixx><ixy>0</ixy><ixz>0</ixz><iyy>0.00001</iyy><iyz>0</iyz><izz>0.00001</izz></inertia></inertial>
@@ -44,7 +73,7 @@
     </link>
     <joint name="lidar_Joint" type="fixed"><parent>base_footprint</parent><child>lidar_frame</child></joint>
-    <link name="depth_cam"><pose>0.061376 -0.00013463 0.121154 0 0 0</pose>
+    <link name="depth_cam"><pose relative_to="fork_mast">${camera_mount_x} ${camera_mount_y} ${camera_mount_z} 0 ${camera_pitch} 0</pose>
       <inertial><mass>0.08</mass><inertia><ixx>0.00002</ixx><ixy>0</ixy><ixz>0</ixz><iyy>0.00002</iyy><iyz>0</iyz><izz>0.00002</izz></inertia></inertial>
-      <visual name="visual"><geometry><box><size>0.045 0.055 0.025</size></box></geometry></visual>
+      <visual name="visual"><pose>0 0 ${-camera_body_height / 2 + camera_mesh_top_z} 0 0 0</pose><geometry><box><size>0.045 0.055 ${camera_body_height}</size></box></geometry></visual>
       <sensor name="depth_camera" type="depth_camera">
         <always_on>true</always_on><update_rate>10</update_rate><visualize>false</visualize>
@@ -54,5 +83,5 @@
       </sensor>
     </link>
-    <joint name="cam_Joint" type="fixed"><parent>base_footprint</parent><child>depth_cam</child></joint>
+    <joint name="cam_Joint" type="fixed"><parent>fork_mast</parent><child>depth_cam</child></joint>
     <link name="imu_link"><pose>0 0 0.07 0 0 0</pose>
       <inertial><mass>0.01</mass><inertia><ixx>0.000001</ixx><ixy>0</ixy><ixz>0</ixz><iyy>0.000001</iyy><iyz>0</iyz><izz>0.000001</izz></inertia></inertial>
@@ -69,4 +98,8 @@
       <frame_id>${robot_name}/odom</frame_id><child_frame_id>${robot_name}/base_footprint</child_frame_id>
     </plugin>
+    <plugin filename="ignition-gazebo-joint-position-controller-system" name="ignition::gazebo::systems::JointPositionController">
+      <joint_name>fork_carriage_joint</joint_name><topic>/${robot_name}/fork/command</topic>
+      <initial_position>0.0</initial_position><p_gain>10</p_gain>
+    </plugin>
   </model>
 </sdf>
