Commit message: feat: 135mm 파렛트와 포크 간극 정합

File: vehicle_simulator_model/ubuntu/ros2_ws/src/mentorpi_description/urdf/mecanum_forklift.urdf (robot description, URDF)
Before this commit: robot mecanum, 15 links, 14 joints
Links:
- link fork_mast: geometry collision box size=0.026 0.02 0.30; collision box size=0.026 0.02 0.30
Joints:
- joint fork_left_joint: origin xyz=0 0.03 0 rpy=0 0 0 -> xyz=0 0.05 -0.007 rpy=0 0 0
- joint fork_right_joint: origin xyz=0 -0.03 0 rpy=0 0 0 -> xyz=0 -0.05 -0.007 rpy=0 0 0

File: vehicle_simulator_model/ubuntu/ros2_ws/src/mentorpi_description/urdf/mecanum_forklift.xacro (robot description, xacro)
@@ -301,5 +301,5 @@
   </link>
   <joint name="fork_left_joint" type="fixed">
-    <origin rpy="0 0 0" xyz="0 0.05 0" />
+    <origin rpy="0 0 0" xyz="0 0.05 -0.007" />
     <parent link="fork_carriage" />
     <child link="fork_left" />
@@ -326,5 +326,5 @@
   </link>
   <joint name="fork_right_joint" type="fixed">
-    <origin rpy="0 0 0" xyz="0 -0.05 0" />
+    <origin rpy="0 0 0" xyz="0 -0.05 -0.007" />
     <parent link="fork_carriage" />
     <child link="fork_right" />

File: vehicle_simulator_model/ubuntu/ros2_ws/src/mentorpi_gz_sim/models/mentorpi_m1/model.sdf.xacro (robot description, xacro)
@@ -92,5 +92,5 @@
     </joint>
     <link name="fork_left">
-      <pose relative_to="fork_carriage">0.09 0.05 0 0 0 0</pose>
+      <pose relative_to="fork_carriage">0.09 0.05 -0.007 0 0 0</pose>
       <inertial><mass>0.03</mass><inertia>
         <ixx>0.00001</ixx><ixy>0</ixy><ixz>0</ixz>
@@ -104,5 +104,5 @@
     <joint name="fork_left_joint" type="fixed"><parent>fork_carriage</parent><child>fork_left</child></joint>
     <link name="fork_right">
-      <pose relative_to="fork_carriage">0.09 -0.05 0 0 0 0</pose>
+      <pose relative_to="fork_carriage">0.09 -0.05 -0.007 0 0 0</pose>
       <inertial><mass>0.03</mass><inertia>
         <ixx>0.00001</ixx><ixy>0</ixy><ixz>0</ixz>
