Commit message: fix(foxglove-assets): serve compatible asset bundle

File: foxglove_assert_server/assets/hiwonder_mecanum_forklift/urdf/hiwonder_mecanum_forklift.urdf (robot description, URDF)
Before this commit: robot hiwonder_mecanum_forklift, 7 links, 6 joints
Links:
- link base_link: geometry visual box size=0.036 0.032 0.010; visual box size=0.085 0.056 0.006
- link lift_mast: geometry visual box size=0.018 0.014 0.28; visual box size=0.018 0.014 0.28
